Commit message: Update arm.urdf

File: j1939_ros_interface/description/arm.urdf (robot description, URDF)
Before this commit: robot arm, 5 links, 4 joints
Links:
- removed link imu
- added link imu1; visual box size=0.5 0.5 0.5
Joints:
- removed joint joint_imu
- added joint joint_imu1: type fixed, parent base, child imu1, origin xyz=0 0 1 rpy=0 0 0, axis 1 0 0
- added joint joint_imu2: type fixed, parent link1, child imu2, origin xyz=0 0 1.5 rpy=0 0 0, axis 1 0 0
